Commit message: feat: Add RGB-D sensor.

File: project4/src/my_robot/urdf/my_robot.xacro (robot description, xacro)
@@ -129,9 +129,9 @@
   <joint type="fixed" name="camera_joint">
     <origin xyz="0.2 0 0" rpy="0 0 0"/>
-    <child link="camera"/>
-    <parent link="chassis"/>
-    <axis xyz="0 1 0" rpy="0 0 0"/>
-  </joint>
-  <link name="camera">
+    <child link="camera_link"/>
+    <parent link="chassis"/>
+    <axis xyz="0 1 0" rpy="0 0 0"/>
+  </joint>
+  <link name="camera_link">
       <collision name='camera_collision'>
         <origin xyz="0 0 0" rpy="0 0 0" />
@@ -181,4 +181,11 @@
     </inertial>
   </link>
+  <joint name="camera_optical_joint" type="fixed">
+    <origin xyz="0 0 0" rpy="-1.5707 0 -1.5707"/>
+    <parent link="camera_link"/>
+    <child link="camera_link_optical"/>
+  </joint>
+  <link name="camera_link_optical">
+  </link>
   <gazebo reference="left_wheel">
     <material>Gazebo/Green</material>
